File: Board/Reactor.sch (KiCad schematic (older format))
At the start: 10 parts, among them P1 CONN_02X13, P2 CONN_01X10, P3 CONN_01X13, P4 CONN_02X04, U1 74LS165

Commit message: _
Connections:
- wire segments 103 -> 105
Changed lines of the file:
@@
 	7000 2750 7200 2750
 Wire Wire Line
-	6200 3400 8200 3400
-Wire Wire Line
-	7050 3400 7050 2850
+	6200 3400 7050 3400
+Wire Wire Line
+	7050 2850 7050 3550
 Wire Wire Line
 	7050 2850 7200 2850
 Wire Wire Line
-	6200 3300 8250 3300
-Wire Wire Line
-	7100 3300 7100 2950
+	6200 3300 7100 3300
+Wire Wire Line
+	7100 2950 7100 3650
 Wire Wire Line
 	7100 2950 7200 2950
@@
 Wire Wire Line
 	7000 2750 7000 3500
-Wire Wire Line
-	8250 3300 8250 4550
-Wire Wire Line
-	8250 4550 7600 4550
-Wire Wire Line
-	8200 3400 8200 4650
-Wire Wire Line
-	8200 4650 7600 4650
 Wire Wire Line
 	8150 3500 8150 4850
@@
 	7750 3850 7750 3700
 Connection ~ 7250 3700
+Wire Wire Line
+	7100 3650 7050 3650
+Wire Wire Line
+	7050 3650 7050 4350
+Wire Wire Line
+	7050 4350 7100 4350
+Wire Wire Line
+	7050 3550 7000 3550
+Wire Wire Line
+	7000 3550 7000 4550
+Wire Wire Line
+	7000 4550 7100 4550
 $EndSCHEMATC

Commit message: Changed to circular board
Parts:
- removed BARREL_JACK: BARREL_JACK, Connect:BARREL_JACK, symbol BARREL_JACK
- added P?: USB_OTG, symbol USB_OTG
Changed lines of the file:
@@
 $EndComp
 $Comp
-L +3V3 #PWR01
+L +3V3 #PWR2
 U 1 1 585C4FF4
 P 4600 1900
-F 0 "#PWR01" H 4600 1750 50  0001 C CNN
+F 0 "#PWR2" H 4600 1750 50  0001 C CNN
 F 1 "+3V3" H 4600 2040 50  0000 C CNN
 F 2 "" H 4600 1900 50  0000 C CNN
@@
 $EndComp
 $Comp
-L GND #PWR02
+L GND #PWR3
 U 1 1 585C5014
 P 4700 5100
-F 0 "#PWR02" H 4700 4850 50  0001 C CNN
+F 0 "#PWR3" H 4700 4850 50  0001 C CNN
 F 1 "GND" H 4700 4950 50  0000 C CNN
 F 2 "" H 4700 5100 50  0000 C CNN
@@
 Text Label 6350 4000 0    60   ~ 0
 D0
-$Comp
-L BARREL_JACK BARREL_JACK
-U 1 1 587B349B
-P 2900 2800
-F 0 "BARREL_JACK" H 2900 3050 50  0000 C CNN
-F 1 "BARREL_JACK" H 2900 2600 50  0000 C CNN
-F 2 "Connect:BARREL_JACK" H 2900 2800 50  0000 C CNN
-F 3 "" H 2900 2800 50  0000 C CNN
-	1    2900 2800
-	1    0    0    -1
-$EndComp
 Wire Wire Line
 	6200 2900 6200 2600
@@
 Connection ~ 6850 4100
 Connection ~ 3650 2700
-Wire Wire Line
-	3200 2800 4000 2800
 Connection ~ 4000 2800
 Wire Wire Line
-	3200 2900 4000 2900
+	2950 2900 4000 2900
 Connection ~ 4000 2900
 $Comp
@@
 $EndComp
 $Comp
-L +5V #PWR03
+L +5V #PWR1
 U 1 1 587B47BB
 P 2050 2100
-F 0 "#PWR03" H 2050 1950 50  0001 C CNN
+F 0 "#PWR1" H 2050 1950 50  0001 C CNN
 F 1 "+5V" H 2050 2240 50  0000 C CNN
 F 2 "" H 2050 2100 50  0000 C CNN
@@
 Text Label 5700 2700 0    60   ~ 0
 ChipEnable
-Wire Wire Line
-	3200 2700 3200 2250
-Wire Wire Line
-	3200 2250 2050 2250
 Connection ~ 2050 2250
 Wire Wire Line
@@
 LED4
 $Comp
-L VCC #PWR?
+L VCC #PWR4
 U 1 1 587FFF48
 P 7900 3850
-F 0 "#PWR?" H 7900 3700 50  0001 C CNN
+F 0 "#PWR4" H 7900 3700 50  0001 C CNN
 F 1 "VCC" H 7900 4000 50  0000 C CNN
 F 2 "" H 7900 3850 50  0000 C CNN
@@
 Wire Wire Line
 	7000 4550 7100 4550
+$Comp
+L USB_OTG P?
+U 1 1 58828F74
+P 2750 1800
+F 0 "P?" H 3075 1675 50  0000 C CNN
+F 1 "USB_OTG" H 2750 2000 50  0000 C CNN
+F 2 "" V 2700 1700 50  0000 C CNN
+F 3 "" V 2700 1700 50  0000 C CNN
+	1    2750 1800
+	1    0    0    -1
+$EndComp
+Wire Wire Line
+	2050 2250 2550 2250
+Wire Wire Line
+	2550 2250 2550 2100
+Wire Wire Line
+	2950 2900 2950 2100
 $EndSCHEMATC
