File: Board/Reactor.sch (KiCad schematic (older format))
At the start: 20 parts, among them P1 CONN_02X13, P2 USER_PORT, P3 CONN_01X13, P4 LA_PWR, P5 USB_OTG, P6 DEBUG, U1 usb1232h, U2 PCF8574

Commit message: - board laid out (draft).
Parts:
- removed D1, D2, D3, D4: LED_Dual_AAC, LEDs_new:LED_D3.0mm-3, symbol LED_Dual_AAC
- removed P4: LA_PWR, Connectors_Molex:Molex_KK-6410-04_04x2.54mm_Straight, symbol CONN_01X04
- removed U1: usb1232h, Housings_DIP:DIP-18_W7.62mm_LongPads, symbol usb1232h
- added D1, D2, D3, D4: LED_Dual_CAC, sip:SIP3, symbol LED_Dual_CAC
- added U1: AdafruitFT232H, ReactorProject:AdafruitFT232h, symbol AdafruitFT232H
Connections:
- net labels removed: +3V3, +5V, VCC
- wire segments 171 -> 140
- no-connect marks 0 -> 26
Other:
- moved on the sheet: P2, P5, R2, R4, R6, R8, U2

Commit message: - Getting PCB ready for manufacture
Parts:
- added U3: SP720APP, dip:DIP16, symbol SP720APP
Connections:
- wire segments 140 -> 160
Changed lines of the file:
@@
 Text Label 7750 4750 0    28   ~ 0
 PA11
+$Comp
+L SP720APP U3
+U 1 1 59026405
+P 7550 2200
+F 0 "U3" H 7550 2200 60  0000 C CNN
+F 1 "SP720APP" H 7550 2200 60  0000 C CNN
+F 2 "dip:DIP16" H 7550 2200 60  0001 C CNN
+F 3 "" H 7550 2200 60  0001 C CNN
+	1    7550 2200
+	0    1    1    0
+$EndComp
 Wire Wire Line
 	5650 4000 9400 4000
@@
 	5700 4300 5200 4300
 Connection ~ 5200 4300
+Wire Wire Line
+	7750 2650 7750 3300
+Connection ~ 7750 3300
+Wire Wire Line
+	7850 2650 7850 3400
+Connection ~ 7850 3400
+Wire Wire Line
+	7950 2650 7950 3500
+Connection ~ 7950 3500
+Wire Wire Line
+	8050 2650 8050 3600
+Connection ~ 8050 3600
+Wire Wire Line
+	8150 2650 8150 3700
+Connection ~ 8150 3700
+Wire Wire Line
+	8250 2650 8250 3800
+Connection ~ 8250 3800
+Wire Wire Line
+	8350 2650 8350 3900
+Connection ~ 8350 3900
+Wire Wire Line
+	8450 1750 8600 1750
+Wire Wire Line
+	8600 1750 8600 2800
+Wire Wire Line
+	8600 2800 8450 2800
+Wire Wire Line
+	8450 2800 8450 4000
+Connection ~ 8450 4000
+Wire Wire Line
+	7750 1750 7400 1750
+Wire Wire Line
+	7400 1750 7400 2450
+Wire Wire Line
+	7400 2450 5200 2450
+Connection ~ 5200 2450
+Wire Wire Line
+	8450 2650 8450 2700
+Wire Wire Line
+	8450 2700 5150 2700
+Connection ~ 5150 2700
+Wire Wire Line
+	6700 2100 6700 2150
+Wire Wire Line
+	6700 2150 5200 2150
+Connection ~ 5200 2150
+Wire Wire Line
+	6750 2100 6750 2200
+Wire Wire Line
+	6750 2200 5100 2200
+Connection ~ 5100 2200
 $EndSCHEMATC

Commit message: Moving to sockets instead of FT232h symbol
Parts:
- removed U1: AdafruitFT232H, ReactorProject:AdafruitFT232h, symbol AdafruitFT232H
- added P4, P8: CONN_01X02, sip:SIP2, symbol CONN_01X02
- added P7, P9: CONN_01X10, Connectors_Molex:Molex_SPOX-5267_22-03-5105_10x2.54mm_Straight, symbol CONN_01X10
Connections:
- wire segments 160 -> 156
- no-connect marks 26 -> 25
Changed lines of the file:
@@
 Text Label 2500 3750 0    28   ~ 0
 USBDP2
-NoConn ~ 6300 1300
-NoConn ~ 6350 1300
-NoConn ~ 6400 1300
-NoConn ~ 6450 1300
-NoConn ~ 6500 1300
-NoConn ~ 6550 1300
-NoConn ~ 6600 1300
-NoConn ~ 6650 1300
-NoConn ~ 6700 1300
-NoConn ~ 6750 1300
 NoConn ~ 7850 5350
 NoConn ~ 8350 5450
@@
 $EndComp
 $Comp
-L AdafruitFT232H U1
-U 1 1 58C47A87
-P 6250 1450
-F 0 "U1" H 6500 1450 28  0000 C CNN
-F 1 "AdafruitFT232H" H 6500 1350 28  0000 C CNN
-F 2 "ReactorProject:AdafruitFT232h" H 6650 1600 28  0001 C CNN
-F 3 "" H 6650 1600 28  0001 C CNN
-	1    6250 1450
-	0    1    1    0
-$EndComp
-$Comp
 L CONN_02X13 P1
 U 1 1 585C4A7F
@@
 Wire Wire Line
 	5650 3700 9400 3700
-Connection ~ 6650 4000
-Connection ~ 6600 3900
-Connection ~ 6550 3800
-Connection ~ 6500 3700
-Connection ~ 6450 3600
-Connection ~ 6400 3500
-Connection ~ 6350 3400
-Connection ~ 6300 3300
 Wire Wire Line
 	8850 4450 10200 4450
@@
 	2450 2300 2450 3750
 Wire Wire Line
-	2450 2300 7350 2300
-Wire Wire Line
-	2500 2350 7300 2350
+	7350 2300 2450 2300
+Wire Wire Line
+	7300 2350 2500 2350
 Wire Wire Line
 	9000 4850 9000 5950
@@
 	9050 6000 4450 6000
 Wire Wire Line
-	7300 2350 7300 1750
-Wire Wire Line
-	7350 2300 7350 1650
-Wire Wire Line
-	7300 1750 7000 1750
-Wire Wire Line
-	7350 1650 7000 1650
-Wire Wire Line
-	6650 4000 6650 2100
-Wire Wire Line
-	6450 3600 6450 2100
-Wire Wire Line
-	6500 3700 6500 2100
-Wire Wire Line
-	6400 3500 6400 2100
+	7300 1650 7300 2350
+Wire Wire Line
+	7350 1600 7350 2300
 Wire Wire Line
 	5650 3600 9400 3600
@@
 	4100 5800 4100 5850
 Wire Wire Line
-	6600 3900 6600 2100
-Wire Wire Line
 	7550 5050 7550 3900
 Connection ~ 7550 3900
@@
 Connection ~ 7200 3600
 Wire Wire Line
-	6550 2100 6550 3800
-Wire Wire Line
 	8350 5550 8650 5550
 Wire Wire Line
@@
 	5650 3300 9400 3300
 Wire Wire Line
-	6350 2100 6350 3150
-Wire Wire Line
-	6350 3150 5750 3150
-Wire Wire Line
-	5750 3150 5750 3400
-Wire Wire Line
-	6300 2100 6300 3100
-Wire Wire Line
-	6300 3100 5700 3100
-Wire Wire Line
-	5700 3100 5700 3300
-Connection ~ 5700 3300
-Wire Wire Line
 	7850 4850 7600 4850
 Wire Wire Line
@@
 	8600 5050 8600 3300
 Connection ~ 8600 3300
-Connection ~ 5750 3400
 Wire Wire Line
 	2300 1800 2300 1900
 Wire Wire Line
-	2300 1900 5200 1900
+	2300 1900 6150 1900
 Wire Wire Line
 	5200 1900 5200 7100
@@
 Connection ~ 5150 2700
 Wire Wire Line
-	6700 2100 6700 2150
-Wire Wire Line
-	6700 2150 5200 2150
-Connection ~ 5200 2150
-Wire Wire Line
-	6750 2100 6750 2200
-Wire Wire Line
-	6750 2200 5100 2200
-Connection ~ 5100 2200
+	3000 1700 3000 1900
+Connection ~ 3000 1900
+Wire Wire Line
+	3100 1700 3100 1950
+Connection ~ 3100 1950
+$Comp
+L CONN_01X02 P4
+U 1 1 5906537A
+P 3050 1500
+F 0 "P4" H 3050 1650 50  0000 C CNN
+F 1 "CONN_01X02" V 3150 1500 50  0000 C CNN
+F 2 "sip:SIP2" H 3050 1500 50  0000 C CNN
+F 3 "" H 3050 1500 50  0000 C CNN
+	1    3050 1500
+	0    -1   -1   0
+$EndComp
+$Comp
+L CONN_01X10 P7
+U 1 1 5908EF0E
+P 6500 1550
+F 0 "P7" H 6500 2100 50  0000 C CNN
+F 1 "CONN_01X10" V 6600 1550 50  0000 C CNN
+F 2 "Connectors_Molex:Molex_SPOX-5267_22-03-5105_10x2.54mm_Straight" H 6500 1550 50  0001 C CNN
+F 3 "" H 6500 1550 50  0000 C CNN
+	1    6500 1550
+	0    -1   -1   0
+$EndComp
+$Comp
+L CONN_01X02 P8
+U 1 1 5908F039
+P 7300 1400
+F 0 "P8" H 7300 1550 50  0000 C CNN
+F 1 "CONN_01X02" V 7400 1400 50  0000 C CNN
+F 2 "sip:SIP2" H 7300 1400 50  0001 C CNN
+F 3 "" H 7300 1400 50  0000 C CNN
+	1    7300 1400
+	0    -1   -1   0
+$EndComp
+Wire Wire Line
+	7300 1650 7250 1650
+Wire Wire Line
+	7250 1650 7250 1600
+Wire Wire Line
+	6050 1750 5100 1750
+Connection ~ 5100 1750
+Wire Wire Line
+	6150 1900 6150 1750
+Connection ~ 5200 1900
+Wire Wire Line
+	6950 1750 6950 3300
+Connection ~ 6950 3300
+Wire Wire Line
+	6850 1750 6850 3400
+Connection ~ 6850 3400
+Wire Wire Line
+	6750 1750 6750 3500
+Connection ~ 6750 3500
+Wire Wire Line
+	6650 1750 6650 3600
+Connection ~ 6650 3600
+Wire Wire Line
+	6550 1750 6550 3700
+Connection ~ 6550 3700
+Wire Wire Line
+	6450 1750 6450 3800
+Connection ~ 6450 3800
+Wire Wire Line
+	6350 1750 6350 3900
+Connection ~ 6350 3900
+Wire Wire Line
+	6250 1750 6250 4000
+Connection ~ 6250 4000
+$Comp
+L CONN_01X10 P9
+U 1 1 59092009
+P 6500 1250
+F 0 "P9" H 6500 1800 50  0000 C CNN
+F 1 "CONN_01X10" V 6600 1250 50  0000 C CNN
+F 2 "Connectors_Molex:Molex_SPOX-5267_22-03-5105_10x2.54mm_Straight" H 6500 1250 50  0001 C CNN
+F 3 "" H 6500 1250 50  0000 C CNN
+	1    6500 1250
+	0    1    1    0
+$EndComp
+NoConn ~ 6950 1050
+NoConn ~ 6850 1050
+NoConn ~ 6750 1050
+NoConn ~ 6650 1050
+NoConn ~ 6550 1050
+NoConn ~ 6450 1050
+NoConn ~ 6350 1050
+NoConn ~ 6250 1050
+NoConn ~ 6150 1050
 $EndSCHEMATC

Commit message: -
Connections:
- net labels removed: D0, D1, D2, D3, D4, D5, D6, D7
Changed lines of the file:
@@
 Comment4 ""
 $EndDescr
-Text Label 6350 3300 0    60   ~ 0
-D7
-Text Label 6350 3400 0    60   ~ 0
-D6
-Text Label 6350 3500 0    60   ~ 0
-D5
-Text Label 6350 3600 0    60   ~ 0
-D4
-Text Label 6350 3700 0    60   ~ 0
-D3
-Text Label 6350 3800 0    60   ~ 0
-D2
-Text Label 6350 3900 0    60   ~ 0
-D1
-Text Label 6350 4000 0    60   ~ 0
-D0
 $Comp
 L R R4
@@
 Text Label 7750 5450 0    28   ~ 0
 PA15
-Text Label 7750 5550 0    28   ~ 0
-PA16
 Text Label 7750 5650 0    28   ~ 0
 PA14
@@
 Connection ~ 5100 3250
 Wire Wire Line
-	7850 5550 7650 5550
-Wire Wire Line
-	7650 5550 7650 3400
-Connection ~ 7650 3400
-Wire Wire Line
 	7850 5750 5200 5750
 Connection ~ 5200 5750
@@
 NoConn ~ 6250 1050
 NoConn ~ 6150 1050
+Text Label 7750 5550 0    28   ~ 0
+PA16
+Wire Wire Line
+	7850 5550 7250 5550
+Wire Wire Line
+	7250 5550 7250 3400
+Connection ~ 7250 3400
 $EndSCHEMATC

Commit message: LEDs are live!
Connections:
- wire segments 156 -> 210
Changed lines of the file:
@@
 $EndComp
 Wire Wire Line
-	5650 4000 9400 4000
-Wire Wire Line
-	5650 3900 9400 3900
-Wire Wire Line
-	5650 3800 9400 3800
-Wire Wire Line
-	5650 3700 9400 3700
+	5650 4000 6250 4000
+Wire Wire Line
+	6250 4000 7400 4000
+Wire Wire Line
+	7400 4000 8450 4000
+Wire Wire Line
+	8450 4000 8750 4000
+Wire Wire Line
+	8750 4000 9400 4000
+Wire Wire Line
+	5650 3900 6350 3900
+Wire Wire Line
+	6350 3900 7450 3900
+Wire Wire Line
+	7450 3900 7550 3900
+Wire Wire Line
+	7550 3900 8350 3900
+Wire Wire Line
+	8350 3900 9400 3900
+Wire Wire Line
+	5650 3800 6450 3800
+Wire Wire Line
+	6450 3800 7500 3800
+Wire Wire Line
+	7500 3800 8250 3800
+Wire Wire Line
+	8250 3800 8650 3800
+Wire Wire Line
+	8650 3800 9400 3800
+Wire Wire Line
+	5650 3700 6550 3700
+Wire Wire Line
+	6550 3700 7350 3700
+Wire Wire Line
+	7350 3700 8150 3700
+Wire Wire Line
+	8150 3700 8700 3700
+Wire Wire Line
+	8700 3700 9400 3700
 Wire Wire Line
 	8850 4450 10200 4450
@@
 	7350 1600 7350 2300
 Wire Wire Line
-	5650 3600 9400 3600
-Wire Wire Line
-	5650 3500 9400 3500
+	5650 3600 6650 3600
+Wire Wire Line
+	6650 3600 7200 3600
+Wire Wire Line
+	7200 3600 8050 3600
+Wire Wire Line
+	8050 3600 8850 3600
+Wire Wire Line
+	8850 3600 9400 3600
+Wire Wire Line
+	5650 3500 6750 3500
+Wire Wire Line
+	6750 3500 7300 3500
+Wire Wire Line
+	7300 3500 7950 3500
+Wire Wire Line
+	7950 3500 8900 3500
+Wire Wire Line
+	8900 3500 9400 3500
 Wire Wire Line
 	2000 6550 2650 6550
@@
 	2100 5200 2100 5050
 Wire Wire Line
-	2100 5050 5150 5050
+	2100 5050 2750 5050
+Wire Wire Line
+	2750 5050 3350 5050
+Wire Wire Line
+	3350 5050 4000 5050
+Wire Wire Line
+	4000 5050 5150 5050
 Wire Wire Line
 	2750 5200 2750 5050
@@
 Connection ~ 8750 4000
 Wire Wire Line
-	5650 3400 9400 3400
-Wire Wire Line
-	5650 3300 9400 3300
+	5650 3400 6850 3400
+Wire Wire Line
+	6850 3400 7250 3400
+Wire Wire Line
+	7250 3400 7600 3400
+Wire Wire Line
+	7600 3400 7850 3400
+Wire Wire Line
+	7850 3400 9400 3400
+Wire Wire Line
+	5650 3300 6950 3300
+Wire Wire Line
+	6950 3300 7750 3300
+Wire Wire Line
+	7750 3300 8550 3300
+Wire Wire Line
+	8550 3300 8600 3300
+Wire Wire Line
+	8600 3300 9400 3300
 Wire Wire Line
 	7850 4850 7600 4850
@@
 	2300 1800 2300 1900
 Wire Wire Line
-	2300 1900 6150 1900
-Wire Wire Line
-	5200 1900 5200 7100
+	2300 1900 3000 1900
+Wire Wire Line
+	3000 1900 5200 1900
+Wire Wire Line
+	5200 1900 6150 1900
+Wire Wire Line
+	5200 1900 5200 2450
+Wire Wire Line
+	5200 2450 5200 3200
+Wire Wire Line
+	5200 3200 5200 4300
+Wire Wire Line
+	5200 4300 5200 5750
+Wire Wire Line
+	5200 5750 5200 5900
+Wire Wire Line
+	5200 5900 5200 7050
+Wire Wire Line
+	5200 7050 5200 7100
 Wire Wire Line
 	7850 4550 5150 4550
 Wire Wire Line
-	5150 1100 5150 7100
+	5150 1100 5150 2700
+Wire Wire Line
+	5150 2700 5150 2950
+Wire Wire Line
+	5150 2950 5150 4550
+Wire Wire Line
+	5150 4550 5150 5050
+Wire Wire Line
+	5150 5050 5150 6050
+Wire Wire Line
+	5150 6050 5150 7100
 Connection ~ 5150 4550
 Wire Wire Line
 	1900 1800 1900 1950
 Wire Wire Line
-	1900 1950 5100 1950
-Wire Wire Line
-	5100 1150 5100 7100
+	1900 1950 3100 1950
+Wire Wire Line
+	3100 1950 5100 1950
+Wire Wire Line
+	5100 1150 5100 1750
+Wire Wire Line
+	5100 1750 5100 1950
+Wire Wire Line
+	5100 1950 5100 3250
+Wire Wire Line
+	5100 3250 5100 7100
 Connection ~ 5100 1950
 Connection ~ 5150 5050
@@
 	2950 7550 2950 7650
 Wire Wire Line
-	2950 7650 4350 7650
+	2950 7650 3050 7650
+Wire Wire Line
+	3050 7650 3150 7650
+Wire Wire Line
+	3150 7650 4350 7650
 Wire Wire Line
 	4350 7650 4350 5900
@@
 	7250 5550 7250 3400
 Connection ~ 7250 3400
+Entry Bus Bus
+	5400 4250 5500 4350
+Entry Bus Bus
+	5400 4250 5500 4350
+Entry Bus Bus
+	5400 4250 5500 4350
+Entry Bus Bus
+	5400 4250 5500 4350
+Entry Bus Bus
+	5400 4250 5500 4350
+Entry Bus Bus
+	5400 4250 5500 4350
+Entry Bus Bus
+	5400 4250 5500 4350
+Entry Bus Bus
+	5400 4250 5500 4350
+Entry Bus Bus
+	5400 4250 5500 4350
+Entry Bus Bus
+	5400 4250 5500 4350
+Entry Bus Bus
+	5400 4250 5500 4350
+Entry Bus Bus
+	5400 4250 5500 4350
+Entry Bus Bus
+	5400 4250 5500 4350
+Entry Bus Bus
+	5400 4250 5500 4350
+Entry Bus Bus
+	5400 4250 5500 4350
+Entry Bus Bus
+	5400 4250 5500 4350
+Entry Bus Bus
+	5400 4250 5500 4350
+Entry Bus Bus
+	5400 4250 5500 4350
+Entry Bus Bus
+	5400 4250 5500 4350
+Entry Bus Bus
+	5400 4250 5500 4350
+Entry Bus Bus
+	5400 4250 5500 4350
+Entry Bus Bus
+	5400 4250 5500 4350
+Entry Bus Bus
+	5400 4250 5500 4350
+Entry Bus Bus
+	5400 4250 5500 4350
+Entry Bus Bus
+	5400 4250 5500 4350
+Entry Bus Bus
+	5400 4250 5500 4350
+Entry Bus Bus
+	5400 4250 5500 4350
+Entry Bus Bus
+	5400 4250 5500 4350
+Entry Bus Bus
+	5400 4250 5500 4350
+Entry Bus Bus
+	5400 4250 5500 4350
+Entry Bus Bus
+	5400 4250 5500 4350
+Entry Bus Bus
+	5400 4250 5500 4350
+Entry Bus Bus
+	5400 4250 5500 4350
+Entry Bus Bus
+	5400 4250 5500 4350
+Entry Bus Bus
+	5400 4250 5500 4350
+Entry Bus Bus
+	6300 4700 6400 4800
+Entry Bus Bus
+	6300 4700 6400 4800
+Entry Bus Bus
+	6300 4700 6400 4800
+Entry Bus Bus
+	6300 4700 6400 4800
+Entry Bus Bus
+	6300 4700 6400 4800
+Entry Bus Bus
+	6300 4700 6400 4800
+Entry Bus Bus
+	6300 4700 6400 4800
+Entry Bus Bus
+	6300 4700 6400 4800
+Entry Bus Bus
+	6300 4700 6400 4800
+Entry Bus Bus
+	6300 4700 6400 4800
+Entry Bus Bus
+	6300 4700 6400 4800
+Entry Bus Bus
+	6300 4700 6400 4800
+Entry Bus Bus
+	6300 4700 6400 4800
 $EndSCHEMATC
