File: Board/Reactor.kicad_pcb (KiCad board)
At the start: 2 copper layers, 72.4 x 77.1 mm, 19 parts, among them P1 CONN_02X13, P2 USER_PORT, P3 CONN_01X13, P5 USB_OTG, P6 DEBUG, U1 AdafruitFT232H, U2 PCF8574

Commit message: - Getting PCB ready for manufacture
Parts:
- added U3: SP720APP, dip:DIP16, F.Cu at (158.8, 127.0)
Connections:
- U1 pad 19: Net-(U1-Pad19) -> /GND
- U1 pad 20: Net-(U1-Pad20) -> /5V
Routing:
- net /5V: track 15.9 -> 96.1 mm
- net /GND: track 170.1 -> 195.8 mm
- net /D4: track 105.9 -> 130.5 mm
- net /D0: track 125.3 -> 108.5 mm, vias 2 -> 3
- net /D1: track 87.5 -> 72.4 mm
- net /D3: track 83.2 -> 97.8 mm
- net /D5: track 115.6 -> 128.9 mm
- net /D7: track 89.5 -> 99.3 mm
- net /D2: track 98.2 -> 105.0 mm
- net /3v3: track 115.7 -> 121.9 mm
- net /D6: track 99.0 -> 100.6 mm
Other:
- board text added: "(May 2017)"
- board text removed: "(March 2017)"

Commit message: Moving to sockets instead of FT232h symbol
Parts:
- removed U1: AdafruitFT232H, ReactorProject:AdafruitFT232h
- added P4: CONN_01X02, sip:SIP2, F.Cu at (174.6, 95.8)
- added P7: CONN_01X10, Connectors_Molex:Molex_SPOX-5267_22-03-5105_10x2.54mm_Straight, F.Cu at (147.6, 105.9)
- added P8: CONN_01X02, Connectors_Terminal_Blocks:TerminalBlock_Pheonix_MPT-2.54mm_2pol, F.Cu at (135.9, 118.4)
- added P9: CONN_01X10, Connectors_Molex:Molex_SPOX-5267_22-03-5105_10x2.54mm_Straight, F.Cu at (127.3, 105.9)
Connections:
- P1 pad 12: /D7 -> /D1
- P1 pad 15: /D3 -> /D1
- P1 pad 18: /D7 -> /D1
- P1 pad 19: /D5 -> /D1
- P1 pad 21: /D6 -> /D1
- P1 pad 22: /D2 -> /D1
- P1 pad 23: /D4 -> /D1
- P1 pad 24: /D3 -> /D1
- P1 pad 3: /D2 -> /D1
- P1 pad 7: /D6 -> /D1
- P2 pad 4: /D2 -> /D1
- P2 pad 5: /D3 -> /D1
- P2 pad 6: /D4 -> /D1
- P2 pad 7: /D5 -> /D1
- P2 pad 8: /D6 -> /D1
- P2 pad 9: /D7 -> /D1
- P6 pad 2: /D5 -> /D1
- P6 pad 3: /D4 -> /D1
- U3 pad 10: /D6 -> /D1
- U3 pad 11: /D5 -> /D1
- U3 pad 12: /D4 -> /D1
- U3 pad 13: /D3 -> /D1
- U3 pad 14: /D2 -> /D1
- U3 pad 9: /D7 -> /D1
Routing:
- net /D1: track 72.4 -> 735.2 mm, vias 1 -> 13
- net /D4: track 130.5 -> 0.00 mm, vias 1 -> 0
- net /D5: track 128.9 -> 0.00 mm, vias 4 -> 0
- net /D2: track 105.0 -> 0.00 mm, vias 1 -> 0
- net /D6: track 100.6 -> 0.00 mm, vias 1 -> 0
- net /D7: track 99.3 -> 0.00 mm, vias 4 -> 0
- net /D3: track 97.8 -> 0.00 mm, vias 1 -> 0
- net /5V: track 96.1 -> 119.8 mm
- net /USBDM2: track 103.8 -> 107.0 mm, vias 0 -> 1
- net /USBDP2: track 102.9 -> 105.7 mm, vias 0 -> 1
- net /GND: track 195.8 -> 197.2 mm
- net /D0: track 108.5 -> 109.2 mm
Other:
- outline, holes or cut-outs redrawn

Commit message: -
Parts:
- added REF**: MountingHole_2.2mm_M2, Mounting_Holes:MountingHole_2.2mm_M2, F.Cu at (138.9, 67.6)
- added REF**: MountingHole_2.2mm_M2, Mounting_Holes:MountingHole_2.2mm_M2, F.Cu at (178.3, 67.6)
- added REF**: MountingHole_2.2mm_M2, Mounting_Holes:MountingHole_2.2mm_M2, F.Cu at (138.9, 123.0)
- added REF**: MountingHole_2.2mm_M2, Mounting_Holes:MountingHole_2.2mm_M2, F.Cu at (178.3, 122.9)
Connections:
- net /D0 renamed /PA0
- P1 pad 11: /D1 -> /PA1
- P1 pad 12: /D1 -> /PA18
- P1 pad 15: /D1 -> /PA13
- P1 pad 18: /D1 -> /PA18
- P1 pad 19: /D1 -> /PA15
- P1 pad 21: /D1 -> /PA16
- P1 pad 22: /D1 -> /PA12
- P1 pad 23: /D1 -> /PA14
- P1 pad 24: /D1 -> /PA13
- P1 pad 3: /D1 -> /PA12
- P1 pad 5: /D1 -> /PA1
- P1 pad 7: /D1 -> /PA16
- P2 pad 3: /D1 -> /PA1
- P2 pad 4: /D1 -> /PA12
- P2 pad 5: /D1 -> /PA13
- P2 pad 6: /D1 -> /PA14
- P2 pad 7: /D1 -> /PA15
- P2 pad 8: /D1 -> /PA16
- P2 pad 9: /D1 -> /PA18
- P6 pad 2: /D1 -> /PA15
- P6 pad 3: /D1 -> /PA14
- P7 pad 10: /D1 -> /PA18
- P7 pad 4: /D1 -> /PA1
- P7 pad 5: /D1 -> /PA12
- P7 pad 6: /D1 -> /PA13
- P7 pad 7: /D1 -> /PA14
- P7 pad 8: /D1 -> /PA15
- P7 pad 9: /D1 -> /PA16
- U3 pad 10: /D1 -> /PA16
- U3 pad 11: /D1 -> /PA15
- U3 pad 12: /D1 -> /PA14
- U3 pad 13: /D1 -> /PA13
- U3 pad 14: /D1 -> /PA12
- U3 pad 15: /D1 -> /PA1
- U3 pad 9: /D1 -> /PA18
Routing:
- net /D1: track 735.2 -> 0.00 mm, vias 13 -> 0
- net /PA14: track 0.00 -> 130.5 mm, vias 0 -> 1
- net /PA15: track 0.00 -> 128.9 mm, vias 0 -> 4
- net /PA12: track 0.00 -> 105.0 mm, vias 0 -> 1
- net /PA16: track 0.00 -> 102.5 mm, vias 0 -> 1
- net /PA18: track 0.00 -> 99.3 mm, vias 0 -> 4
- net /PA13: track 0.00 -> 97.8 mm, vias 0 -> 1
- net /PA1: track 0.00 -> 86.7 mm, vias 0 -> 1
- net /3v3: track 121.9 -> 128.8 mm

Commit message: -
Routing:
- net /PA14: track 130.5 -> 123.4 mm
- net /PA15: track 128.9 -> 131.3 mm
- net /USBDP2: track 105.7 -> 103.6 mm
- net /PA1: track 86.7 -> 87.7 mm
- net /5V: track 119.8 -> 118.8 mm

Commit message: Generated Gerbers for next spin
Parts:
- moved P8 7.25 mm to (143.0, 119.8), turned to 90 degrees
Routing:
- net /USBDM2: track 107.0 -> 113.1 mm
- net /USBDP2: track 103.6 -> 105.3 mm
- net /PA0: track 109.2 -> 109.8 mm
Other:
- board text added: "(June 2017)"
- board text removed: "(May 2017)"
